Commit message: eoh

File: uuv_descriptions/models/rexrov/urdf/rexrov_sensors.xacro (robot description, xacro)
@@ -39,5 +39,5 @@
   <!-- Mount a camera -->
   <xacro:default_camera namespace="${namespace}" parent_link="${namespace}/base_link" suffix="">
-    <origin xyz="1.15 0 0.4" rpy="0 0.6 0"/>
+    <origin xyz="1.15 0 0.4" rpy="0 0 0"/>
   </xacro:default_camera>
   <xacro:default_camera namespace="${namespace}" parent_link="${namespace}/base_link" suffix="right">
